Commit message: added wsg-50 gripper

File: robots/herb.urdf.xacro (robot description, xacro)
@@ -3,4 +3,5 @@
   <xacro:include filename="bh280.urdf.xacro"/>
   <xacro:include filename="bh282.urdf.xacro"/>
+  <xacro:include filename="weiss_fmf.urdf.xacro"/>
   <xacro:include filename="wam.urdf.xacro"/>
   <xacro:include filename="fixed_transforms.urdf.xacro"/>
@@ -8,5 +9,5 @@
        optionally the BH-280 BarrettHand end-effector. -->
   <xacro:macro name="herb_manipulator"
-               params="prefix:=${prefix} bh280:=false bh282:=false">
+               params="prefix:=${prefix} bh280:=false bh282:=false weiss_fmf:=false">
     <xacro:wam prefix="${prefix}"/>
     <xacro:if value="${bh280}">
@@ -15,4 +16,7 @@
     <xacro:if value="${bh282}">
       <xacro:bh282 prefix="${prefix}"/>
+    </xacro:if>
+    <xacro:if value="${weiss_fmf}">
+      <xacro:weiss_fmf prefix="${prefix}"/>
     </xacro:if>
     <link name="${prefix}/force_torque">
@@ -48,4 +52,12 @@
       </joint>
     </xacro:if>
+  <xacro:if value="${weiss_fmf}">
+      <joint name="${prefix}/hand_mount" type="fixed">
+        <!-- The force/torque sensor is 12 mm thick. -->
+        <origin xyz="0 0 0.012" rpy="0 0 ${pi/2}"/>
+        <parent link="${prefix}/force_torque"/>
+        <child link="${prefix}/hand_base"/>
+      </joint>
+    </xacro:if>
   </xacro:macro>
   <!-- hand arguments should all default to false to make argument passing sane -->
@@ -54,6 +66,8 @@
   <xacro:arg name="left_bh282" default="false"/>
   <xacro:arg name="right_bh282" default="false"/>
-  <xacro:herb_manipulator prefix="/left" bh280="$(arg left_bh280)" bh282="$(arg left_bh282)"/>
-  <xacro:herb_manipulator prefix="/right" bh280="$(arg right_bh280)" bh282="$(arg right_bh282)"/>
+  <xacro:arg name="left_weiss_fmf" default="false"/>
+  <xacro:arg name="right_weiss_fmf" default="false"/>
+  <xacro:herb_manipulator prefix="/left" bh280="$(arg left_bh280)" bh282="$(arg left_bh282)" weiss_fmf="$(arg left_weiss_fmf)"/>
+  <xacro:herb_manipulator prefix="/right" bh280="$(arg right_bh280)" bh282="$(arg right_bh282)" weiss_fmf="$(arg right_weiss_fmf)"/>
   <xacro:herb_base prefix=""/>
   <joint name="/left/wam_mount" type="fixed">
